Commit message: Fix AMP coord-frame bug + widen URDF leg limits + add multi-clip prep
The big finding: 14 AMP training runs (r1-r14) chronically saw
style_r/step ≈ 0.002 because the .npy reference's `root_position`
advanced along world +X with a constant Rx(-90°) `root_quaternion`,
which after AMPLoader's `R.T @ v_world` transform put expert forward
velocity at body +X — but the policy's runtime base-frame velocity
sits at body -Z. The discriminator decided expert-vs-policy off this
constant 3-vector mismatch and ignored everything else.

Fixed in tools/convert_unity_anim_to_npy.py:418-434 (now writes along
world -Y matching the post-spawn-rotation deer-forward direction) and
applied in-place to deer_walk.npy + deer_run.npy via the new
tools/patch_walk_npy_axis.py. After the fix, r15 produced style_r 0.39
in 3000 iters — a 130x jump that finally trained a real walking policy.

Also widened the URDF/USD leg joint limits (fetlock ±28.6° -> ±68.8°,
hip ±45.8° -> ±80.2°, knee 103° -> 126°) because pre-widening
22/31 walk frames clamped front fetlock and 11/12 leg joints clamped
on run.npy — flat-footing the AMP reference. Walk reference clamping
went 71% -> 19% on the worst joint after re-conversion. r19 trained
through 3000 iters with the widened limits using the defensive layers
below.

Hardened PhysX + added defensive guards because widened limits gave
the policy more chances to drive joint state into NaN territory:
- max_linear_velocity 1000 -> 50, max_angular_velocity 1000 -> 20
  (Isaac Lab quadruped boilerplate defaults were unrealistic and let
  PhysX yank self-colliding bodies apart at NaN-inducing speeds)
- solver_position_iteration_count 8 -> 16, velocity 0 -> 2
- Zeroed dof_acc_l2 and dof_torques_l2 weights in V11 env (their
  tiny weights overflowed to -inf when joint state spiked, cascading
  to RuntimeError: normal expects all elements of std >= 0.0)
- Defensive std_param clamp + non-finite guard in train_amp.py as
  a belt-and-braces backstop

New tooling:
- tools/render_playback_video.py — stick-figure offline renderer
- tools/render_playback_meshed.py — full deer-mesh offline renderer
  via trimesh + matplotlib 3D, sidesteps the broken Isaac Sim viewer
  (omni.hydra.rtx crashes on RTX 50-series + Isaac Sim 5.1)
- tools/import_world_urdf_v3.py — URDF->USD regen (had to bypass via
  direct pxr edit instead because the importer pulls in the broken
  RTX renderer; left in tree for when that's fixed upstream)
- play_amp.py: --realtime flag (paces 50 Hz so viewer is watchable;
  earlier "viewer crashes" were actually <2 sec invisible runs) and
  --video flag (dumps trajectory .npz to render offline)

New env classes + tasks:
- DeerUsdWalkAMPEnvCfgV10 / AMP-v13: lower action_rate_l2 (turned out
  to not be the bottleneck — caused noise_std drift instead)
- DeerUsdWalkAMPEnvCfgV11 / AMP-v14: zeroed L2 smoothness penalties,
  the config that finally trained 3000 iters cleanly with widened
  limits in r19

Co-Authored-By: Claude Opus 4.7 (1M context) <noreply@anthropic.com>

File: assets/deer_urdf/deer_world.urdf (robot description, URDF)
Before this commit: robot deer, 16 links, 15 joints
Joints:
- joint FL_shin_to_FL_foot: limit lower=-0.5 upper=0.5 effort=60.0 velocity=10.0 -> lower=-1.2 upper=1.2 effort=60.0 velocity=10.0
- joint FL_thigh_to_FL_shin: limit lower=0.0 upper=1.8 effort=80.0 velocity=10.0 -> lower=0.0 upper=2.2 effort=80.0 velocity=10.0
- joint FR_shin_to_FR_foot: limit lower=-0.5 upper=0.5 effort=60.0 velocity=10.0 -> lower=-1.2 upper=1.2 effort=60.0 velocity=10.0
- joint FR_thigh_to_FR_shin: limit lower=0.0 upper=1.8 effort=80.0 velocity=10.0 -> lower=0.0 upper=2.2 effort=80.0 velocity=10.0
- joint HL_shin_to_HL_foot: limit lower=-0.5 upper=0.5 effort=60.0 velocity=10.0 -> lower=-1.2 upper=1.2 effort=60.0 velocity=10.0
- joint HL_thigh_to_HL_shin: limit lower=-1.8 upper=0.0 effort=80.0 velocity=10.0 -> lower=-2.2 upper=0.0 effort=80.0 velocity=10.0
- joint HR_shin_to_HR_foot: limit lower=-0.5 upper=0.5 effort=60.0 velocity=10.0 -> lower=-1.2 upper=1.2 effort=60.0 velocity=10.0
- joint HR_thigh_to_HR_shin: limit lower=-1.8 upper=0.0 effort=80.0 velocity=10.0 -> lower=-2.2 upper=0.0 effort=80.0 velocity=10.0
- joint chest_to_FL_thigh: limit lower=-0.8 upper=0.8 effort=100.0 velocity=10.0 -> lower=-1.4 upper=1.4 effort=100.0 velocity=10.0
- joint chest_to_FR_thigh: limit lower=-0.8 upper=0.8 effort=100.0 velocity=10.0 -> lower=-1.4 upper=1.4 effort=100.0 velocity=10.0
- joint pelvis_to_HL_thigh: limit lower=-0.8 upper=0.8 effort=100.0 velocity=10.0 -> lower=-1.4 upper=1.4 effort=100.0 velocity=10.0
- joint pelvis_to_HR_thigh: limit lower=-0.8 upper=0.8 effort=100.0 velocity=10.0 -> lower=-1.4 upper=1.4 effort=100.0 velocity=10.0

Commit message: Widen torso joints + prep multi-clip AMP configs
URDF + USD torso joint limits widened (paired with reconverted .npy):
- pelvis_to_chest: ±0.2 -> ±0.5 rad   (±28.6°, was ±11.5°)
- chest_to_neck:  -0.3/+0.5 -> -0.6/+0.8 rad (-34/+46°)
- neck_to_skull:  -0.4/+0.6 -> -0.8/+0.8 rad (±46°)

User feedback on r19's mesh playback was that hips swung more but the
WHOLE BODY was stiff — knees barely moved, spine/neck/head locked.
Tracking this back: idle.npy clamped pelvis_to_chest 68/331 frames at
the prior ±11.5° limit; real deer flex spine ~30°+ in gait. Walk.npy's
torso amplitudes are tiny (2.4° at pelvis_to_chest) — single-clip walk
won't drive much spine motion regardless. Multi-clip is the bigger lever.

New configs ready for r21+:
- DEER_USD_AMP_WALK_RUN_CFG  : walk + run two-clip AMP dataset
- DEER_USD_AMP_WALK_RUN_IDLE_CFG: walk + run + idle three-clip
- DeerUsdWalkAMPEnvCfgV12: V11 + wider velocity range (0.3-2.5 m/s)
  to span both gait speeds in the dataset
- AMP-v15 task: V12 env + walk+run dataset
- AMP-v16 task: V12 env + walk+run+idle dataset

r20 = torso-only widening with single walk clip (running now); r21 will
test multi-clip; r22 combines.

Co-Authored-By: Claude Opus 4.7 (1M context) <noreply@anthropic.com>

File: assets/deer_urdf/deer_world.urdf (robot description, URDF)
Before this commit: robot deer, 16 links, 15 joints
Joints:
- joint chest_to_neck: limit lower=-0.3 upper=0.5 effort=50.0 velocity=8.0 -> lower=-0.6 upper=0.8 effort=50.0 velocity=8.0
- joint neck_to_skull: limit lower=-0.4 upper=0.6 effort=30.0 velocity=8.0 -> lower=-0.8 upper=0.8 effort=30.0 velocity=8.0
- joint pelvis_to_chest: limit lower=-0.2 upper=0.2 effort=120.0 velocity=8.0 -> lower=-0.5 upper=0.5 effort=120.0 velocity=8.0

Commit message: Add the polyart deer: AMP/ASE training, rig pipeline and evaluation
The 38-joint deer built from the Malbers model, and everything used to train and judge it:

- training/polyart: environment, rewards, hoof observations, ASE stage 1 with the
  diversity objective
- tools/rig_pipeline: URDF build, FK-validated reference extraction, preflight checks,
  gait reports, rollout collection, z-sweeps
- tools: matched-condition evaluation (load share, hoof slip, ankle contact, stride
  regularity) and phase-aligned ASE skill separation, with CPU tests for the ASE and
  hoof-channel wiring
- experiments/launch: the exact configuration of every training run, plus a tag-to-run map
- docs: write-ups of each finding, including the 1.25x reference scale bug

Co-Authored-By: Claude Opus 5.5 <noreply@anthropic.com>

File: assets/deer_urdf/deer_world.urdf (robot description, URDF)
Before this commit: robot deer, 16 links, 15 joints
Links:
- added link FL_hip_abd, mass 0.001
- added link FL_toe, mass 0.25; collision mesh filename=meshes/world/FL_toe_collision.stl
- added link FR_hip_abd, mass 0.001
- added link FR_toe, mass 0.25; collision mesh filename=meshes/world/FR_toe_collision.stl
- added link HL_hip_abd, mass 0.001
- added link HL_toe, mass 0.25; collision mesh filename=meshes/world/HL_toe_collision_fixed.stl
- added link HR_hip_abd, mass 0.001
- added link HR_toe, mass 0.25; collision mesh filename=meshes/world/HR_toe_collision_fixed.stl
- added link antlers, mass 1.5; collision mesh filename=meshes/world/antler_collision_v2.stl
- added link chest_yaw_link, mass 0.001
- added link neck_yaw_link, mass 0.001
- link FL_foot: mass 1.0 -> 0.55
- link FL_shin: mass 1.5 -> 1.7
- link FL_thigh: mass 2.5 -> 3.0
- link FR_foot: mass 1.0 -> 0.55
- link FR_shin: mass 1.5 -> 1.7
- link FR_thigh: mass 2.5 -> 3.0
- link HL_foot: mass 0.8 -> 0.55
- link HL_shin: mass 1.0 -> 1.7
- link HL_thigh: mass 1.2 -> 2.5
- link HR_foot: mass 0.8 -> 0.55
- link HR_shin: mass 1.0 -> 1.7
- link HR_thigh: mass 1.2 -> 2.5
- link chest: mass 28.0 -> 41.5
- link neck: mass 6.0 -> 5.0
- link pelvis: mass 18.0 -> 10.0
- link skull: mass 5.0 -> 3.0; geometry collision mesh filename=meshes/world/skull_collision_v2.stl; visual mesh filename=meshes/world/skull_visual.stl
Joints:
- removed joint chest_to_FL_thigh
- removed joint chest_to_FR_thigh
- removed joint chest_to_neck
- removed joint pelvis_to_HL_thigh
- removed joint pelvis_to_HR_thigh
- removed joint pelvis_to_chest
- added joint FL_foot_to_FL_toe: type revolute, parent FL_foot, child FL_toe, origin xyz=-0.003615 -0.046036 -0.271656 rpy=0 0 0, axis 1 0 0, limit lower=-0.400000 upper=1.200000 effort=50.0 velocity=10.0
- added joint FL_hipabd_to_FL_thigh: type revolute, parent FL_hip_abd, child FL_thigh, origin xyz=0 0 0 rpy=0 0 0, axis 1 0 0, limit lower=-1.4 upper=1.4 effort=100.0 velocity=10.0
- added joint FR_foot_to_FR_toe: type revolute, parent FR_foot, child FR_toe, origin xyz=0.003615 -0.046036 -0.271656 rpy=0 0 0, axis 1 0 0, limit lower=-0.400000 upper=1.200000 effort=50.0 velocity=10.0
- added joint FR_hipabd_to_FR_thigh: type revolute, parent FR_hip_abd, child FR_thigh, origin xyz=0 0 0 rpy=0 0 0, axis 1 0 0, limit lower=-1.4 upper=1.4 effort=100.0 velocity=10.0
- added joint HL_foot_to_HL_toe: type revolute, parent HL_foot, child HL_toe, origin xyz=-0.008378 -0.058986 -0.333707 rpy=0 0 0, axis 1 0 0, limit lower=-0.400000 upper=1.200000 effort=50.0 velocity=10.0
- added joint HL_hipabd_to_HL_thigh: type revolute, parent HL_hip_abd, child HL_thigh, origin xyz=0 0 0 rpy=0 0 0, axis 1 0 0, limit lower=-1.4 upper=1.4 effort=100.0 velocity=10.0
- added joint HR_foot_to_HR_toe: type revolute, parent HR_foot, child HR_toe, origin xyz=0.008378 -0.058986 -0.333707 rpy=0 0 0, axis 1 0 0, limit lower=-0.400000 upper=1.200000 effort=50.0 velocity=10.0
- added joint HR_hipabd_to_HR_thigh: type revolute, parent HR_hip_abd, child HR_thigh, origin xyz=0 0 0 rpy=0 0 0, axis 1 0 0, limit lower=-1.4 upper=1.4 effort=100.0 velocity=10.0
- added joint chest_to_FL_hipabd: type revolute, parent chest, child FL_hip_abd, origin xyz=0.121934 0.215348 -0.471727 rpy=0 0 0, axis 0 0 1, limit lower=-0.4 upper=0.4 effort=100.0 velocity=10.0
- added joint chest_to_FR_hipabd: type revolute, parent chest, child FR_hip_abd, origin xyz=-0.122050 0.215239 -0.471956 rpy=0 0 0, axis 0 0 1, limit lower=-0.4 upper=0.4 effort=100.0 velocity=10.0
- added joint chest_to_neck_yaw: type revolute, parent chest, child neck_yaw_link, origin xyz=0.000008 0.004488 -0.426567 rpy=0 0 0, axis 0 1 0, limit lower=-1.500000 upper=1.500000 effort=50.0 velocity=8.0
- added joint chest_yaw_to_chest: type revolute, parent chest_yaw_link, child chest, origin xyz=0 0 0 rpy=0 0 0, axis 1 0 0, limit lower=-0.700000 upper=0.700000 effort=120.0 velocity=8.0
- added joint neck_yaw_to_neck: type revolute, parent neck_yaw_link, child neck, origin xyz=0 0 0 rpy=0 0 0, axis 1 0 0, limit lower=-1.600000 upper=1.600000 effort=50.0 velocity=8.0
- added joint pelvis_to_HL_hipabd: type revolute, parent pelvis, child HL_hip_abd, origin xyz=0.127008 0.189755 0.187934 rpy=0 0 0, axis 0 0 1, limit lower=-0.4 upper=0.4 effort=100.0 velocity=10.0
- added joint pelvis_to_HR_hipabd: type revolute, parent pelvis, child HR_hip_abd, origin xyz=-0.127008 0.189755 0.187936 rpy=0 0 0, axis 0 0 1, limit lower=-0.4 upper=0.4 effort=100.0 velocity=10.0
- added joint pelvis_to_chest_yaw: type revolute, parent pelvis, child chest_yaw_link, origin xyz=-0.000001 0.011858 -0.177186 rpy=0 0 0, axis 0 1 0, limit lower=-0.500000 upper=0.500000 effort=120.0 velocity=8.0
- added joint skull_to_antlers: type fixed, parent skull, child antlers, origin xyz=0 0 0 rpy=0 0 0
- joint FL_shin_to_FL_foot: limit lower=-1.2 upper=1.2 effort=60.0 velocity=10.0 -> lower=-0.300000 upper=1.600000 effort=60.0 velocity=10.0
- joint FR_shin_to_FR_foot: limit lower=-1.2 upper=1.2 effort=60.0 velocity=10.0 -> lower=-0.300000 upper=1.600000 effort=60.0 velocity=10.0
- joint HL_shin_to_HL_foot: limit lower=-1.2 upper=1.2 effort=60.0 velocity=10.0 -> lower=-1.600000 upper=0.300000 effort=60.0 velocity=10.0
- joint HR_shin_to_HR_foot: limit lower=-1.2 upper=1.2 effort=60.0 velocity=10.0 -> lower=-1.600000 upper=0.300000 effort=60.0 velocity=10.0
- joint neck_to_skull: limit lower=-0.8 upper=0.8 effort=30.0 velocity=8.0 -> lower=-1.000000 upper=1.000000 effort=30.0 velocity=8.0
